File: EAGLE_Schematic/switch_board.sch (EAGLE design)
At the start: 90 parts, among them IC1 LM1117MPX-5.0, J1 POWER_JACKPTH, Q1 BC847SMD

Commit message: Fixed a text
Other:
- note added: "VIDEO SWITCH WITH 8 INPUTS AND 1 OUTPUT (MOD. JL-1701) SCART: AUDIO L+R, RGB, COMPOSITE, ASPECT RATIO, BLANKING COMPONENT: AUDIO L+R, Y Pb/Cb Pr/Cr TESTED UP TO 1080p COPYRIGHT (c) 2017-2018 JACKSOFT LABS"
- note removed: "VIDEO SWITCH WITH 8 INPUTS AND 1 OUTPUT (MOD. JL-1701) SCART: AUDIO L+R, RGB, COMPOSITE, ASPECT RATIO, BLANKING COMPONENT: AUDIO L+R, Y Pb/Cb Pr/Cr TESTED UP TO 1080p"
Changed lines of the file:
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@@
 <text x="-233.68" y="96.52" size="1.778" layer="91">FOR MUX CHIPS</text>
 <text x="-160.02" y="96.52" size="1.778" layer="91">FOR PIC</text>
-<text x="-200.66" y="127" size="1.778" layer="91">VIDEO SWITCH WITH 8 INPUTS AND 1 OUTPUT (MOD. JL-1701)
+<text x="-200.66" y="121.92" size="1.778" layer="91">VIDEO SWITCH WITH 8 INPUTS AND 1 OUTPUT (MOD. JL-1701)
 SCART: AUDIO L+R, RGB, COMPOSITE, ASPECT RATIO, BLANKING
-COMPONENT: AUDIO L+R, Y Pb/Cb Pr/Cr TESTED UP TO 1080p</text>
+COMPONENT: AUDIO L+R, Y Pb/Cb Pr/Cr TESTED UP TO 1080p
+COPYRIGHT (c) 2017-2018 JACKSOFT LABS</text>
 </plain>
 <instances>
